File: HB-UNI-SEN-PCB/HB-UNI-SEN-PCB.kicad_pcb (KiCad board)
At the start: 2 copper layers, 44.4 x 30.5 mm, 17 parts, among them J0 BATT, J1 I2C_1, J2 I2C_2, J3 A0, J4 A1, J5 A2, J6 A3, J7 PROG, SW1 CONFIG_BUTTON, U1 ArduinoProMini, U2 CC1101

Commit message: Added new PCB HB-UNI-644, removed unfinished HB-UNI-SEN-O
Other:
- board text added: "Version 1.3 - 05/2018"
- board text removed: "Version 1.2 - 04/2018"

Commit message: Relicened under CC BY-ND-SA
Parts:
- added G***: LOGO, Homebrew:CC-BY-ND-SA, B.Cu at (139.7, 56.5)
Other:
- board text added: "Version 1.4 - 08/2018"
- board text removed: "Version 1.3 - 05/2018"
