File: HB-UNI-SEN-PCB/HB-UNI-SEN-PCB.sch (KiCad schematic (older format))
At the start: 15 parts, among them J0 BATT, J1 I2C_1, J2 I2C_2, J3 A0, J4 A1, J5 A2, J6 A3, J7 PROG, SW1 CONFIG_BUTTON, U1 ArduinoProMini, U2 CC1101

Commit message: Added new PCB HB-UNI-644, removed unfinished HB-UNI-SEN-O
Parts:
- U2: symbol CC1101 -> CC1101-RESCUE-HB-UNI-SEN-PCB
Connections:
- no-connect marks 5 -> 7
Changed lines of the file:
@@
 EESchema Schematic File Version 2
+LIBS:HB-UNI-SEN-PCB-rescue
 LIBS:power
 LIBS:device
@@
 $EndComp
 $Comp
-L CC1101 U2
+L CC1101-RESCUE-HB-UNI-SEN-PCB U2
 U 1 1 5AC3AFA1
 P 1650 5900
@@
 Wire Wire Line
 	2600 3700 2900 3700
-Wire Wire Line
-	2600 3900 2900 3900
 $Comp
 L GND #PWR013
@@
 	4350 2500 4800 2500
 Connection ~ 4700 2500
-$Comp
-L ArduinoProMini U1
-U 1 1 5ACA0010
-P 1900 3100
-F 0 "U1" H 1400 4450 60  0000 C CNN
-F 1 "ArduinoProMini" H 2050 2200 60  0000 C CNN
-F 2 "Homebrew:ArduinoProMini" H 1900 3000 60  0001 C CNN
-F 3 "" H 1900 3000 60  0001 C CNN
-	1    1900 3100
-	1    0    0    -1
-$EndComp
 $Comp
 L PWR_FLAG #FLG014
@@
 Wire Wire Line
 	2600 3600 2900 3600
-Text Label 2700 3900 0    60   ~ 0
+Text Label 2700 4100 0    60   ~ 0
 RSET
 Text Label 2600 5350 0    60   ~ 0
@@
 Wire Wire Line
 	6200 1150 7150 1150
+$Comp
+L ArduinoProMini U1
+U 1 1 5AF60EC1
+P 1900 3100
+F 0 "U1" H 1400 4450 60  0000 C CNN
+F 1 "ArduinoProMini" H 2050 1950 60  0000 C CNN
+F 2 "Homebrew:ArduinoProMini" H 1900 3000 60  0001 C CNN
+F 3 "" H 1900 3000 60  0001 C CNN
+	1    1900 3100
+	1    0    0    -1
+$EndComp
+Wire Wire Line
+	2600 4100 2900 4100
+NoConn ~ 2600 3800
+NoConn ~ 2600 3900
 $EndSCHEMATC

Commit message: * Switched to Kicad 5 * Added HB-UNI-644-S4-A4 addon Board
Parts:
- D1: symbol LED -> Device:LED
- J0, J5, J6: symbol Conn_01x02 -> conn:Conn_01x02
- J1, J2, J7: symbol Conn_01x04 -> conn:Conn_01x04
- J3, J4: symbol Conn_01x03 -> conn:Conn_01x03
- R1, R2, R3: symbol R -> Device:R
- SW1: symbol SW_DIP_x01 -> switches:SW_DIP_x01
- U1: symbol ArduinoProMini -> Homebrew:ArduinoProMini
- U2: symbol CC1101-RESCUE-HB-UNI-SEN-PCB -> HB-UNI-SEN-PCB-rescue:CC1101-RESCUE-HB-UNI-SEN-PCB
Connections:
- wire segments 62 -> 73
Changed lines of the file:
@@
-EESchema Schematic File Version 2
-LIBS:HB-UNI-SEN-PCB-rescue
-LIBS:power
-LIBS:device
-LIBS:switches
-LIBS:relays
-LIBS:motors
-LIBS:transistors
-LIBS:conn
-LIBS:linear
-LIBS:regul
-LIBS:74xx
-LIBS:cmos4000
-LIBS:adc-dac
-LIBS:memory
-LIBS:xilinx
-LIBS:microcontrollers
-LIBS:dsp
-LIBS:microchip
-LIBS:analog_switches
-LIBS:motorola
-LIBS:texas
-LIBS:intel
-LIBS:audio
-LIBS:interface
-LIBS:digital-audio
-LIBS:philips
-LIBS:display
-LIBS:cypress
-LIBS:siliconi
-LIBS:opto
-LIBS:atmel
-LIBS:contrib
-LIBS:valves
-LIBS:Homebrew
+EESchema Schematic File Version 4
 LIBS:HB-UNI-SEN-PCB-cache
-EELAYER 25 0
+EELAYER 26 0
 EELAYER END
 $Descr A4 11693 8268
@@
 $EndDescr
 $Comp
-L Conn_01x04 J1
+L conn:Conn_01x04 J1
 U 1 1 5ABE0D25
 P 6750 1050
@@
 $EndComp
 $Comp
-L Conn_01x04 J2
+L conn:Conn_01x04 J2
 U 1 1 5ABE0DC1
 P 7350 1050
@@
 $EndComp
 $Comp
-L SW_DIP_x01 SW1
+L switches:SW_DIP_x01 SW1
 U 1 1 5ABE0E28
 P 4050 2500
@@
 $EndComp
 $Comp
-L LED D1
+L Device:LED D1
 U 1 1 5ABE1195
 P 4200 2000
@@
 $EndComp
 $Comp
-L +3.3V #PWR01
+L power:+3.3V #PWR01
 U 1 1 5ABE128D
 P 950 1900
@@
 $EndComp
 $Comp
-L Conn_01x03 J3
+L conn:Conn_01x03 J3
 U 1 1 5ABE1EB3
 P 7350 2350
@@
 $EndComp
 $Comp
-L Conn_01x03 J4
+L conn:Conn_01x03 J4
 U 1 1 5ABE1F38
 P 7350 3200
@@
 $EndComp
 $Comp
-L Conn_01x02 J5
+L conn:Conn_01x02 J5
 U 1 1 5ABE1F9E
 P 7350 3800
@@
 $EndComp
 $Comp
-L Conn_01x02 J6
+L conn:Conn_01x02 J6
 U 1 1 5ABE2007
 P 7350 4450
@@
 $EndComp
 $Comp
-L R R1
+L Device:R R1
 U 1 1 5ABE25C7
 P 3650 2000
@@
 $EndComp
 $Comp
-L R R2
+L Device:R R2
 U 1 1 5ABE27F2
 P 6900 1950
@@
 $EndComp
 $Comp
-L R R3
+L Device:R R3
 U 1 1 5ABE28D1
 P 6900 2800
@@
 $EndComp
 $Comp
-L Conn_01x02 J0
+L conn:Conn_01x02 J0
 U 1 1 5ABE2E32
 P 1650 900
@@
 $EndComp
 $Comp
-L CC1101-RESCUE-HB-UNI-SEN-PCB U2
+L HB-UNI-SEN-PCB-rescue:CC1101-RESCUE-HB-UNI-SEN-PCB U2
 U 1 1 5AC3AFA1
 P 1650 5900
@@
 $EndComp
 $Comp
-L Conn_01x04 J7
+L conn:Conn_01x04 J7
 U 1 1 5AC3B268
 P 7350 5300
@@
 	950  1900 1150 1900
 $Comp
-L +3.3V #PWR02
+L power:+3.3V #PWR02
 U 1 1 5AC7DE60
 P 6000 950
@@
 $EndComp
 $Comp
-L GND #PWR03
+L power:GND #PWR03
 U 1 1 5AC7DE98
 P 6000 1050
@@
 $EndComp
 Wire Wire Line
-	6000 950  7150 950
+	6000 950  6550 950
 Connection ~ 6550 950
 Wire Wire Line
-	6000 1050 7150 1050
+	6000 1050 6550 1050
 Connection ~ 6550 1050
 Wire Wire Line
-	6200 1250 7150 1250
+	6200 1250 6550 1250
 Connection ~ 6550 1250
 Connection ~ 6550 1150
 $Comp
-L +3.3V #PWR04
+L power:+3.3V #PWR04
 U 1 1 5AC7EBE5
 P 900 900
@@
 $EndComp
 $Comp
-L GND #PWR05
+L power:GND #PWR05
 U 1 1 5AC7ECC2
 P 900 1000
@@
 $EndComp
 Wire Wire Line
-	900  900  1450 900
+	900  900  1250 900
 Wire Wire Line
 	900  1000 1450 1000
 $Comp
-L GND #PWR06
+L power:GND #PWR06
 U 1 1 5AC7F222
 P 6650 2350
@@
 $EndComp
 $Comp
-L +3.3V #PWR07
+L power:+3.3V #PWR07
 U 1 1 5AC7F4EE
 P 1200 5350
@@
 	1200 5350 1350 5350
 $Comp
-L GND #PWR08
+L power:GND #PWR08
 U 1 1 5AC7FA89
 P 1200 5900
@@
 	1200 5900 1350 5900
 $Comp
-L GND #PWR09
+L power:GND #PWR09
 U 1 1 5AC7FD3C
 P 950 3750
@@
 $EndComp
 Wire Wire Line
-	950  3700 1150 3700
+	950  3700 1050 3700
 Wire Wire Line
 	950  3750 950  3700
@@
 	6900 2450 7150 2450
 Wire Wire Line
-	6900 2250 7150 2250
-Wire Wire Line
-	6650 2350 7150 2350
+	6900 2250 7100 2250
+Wire Wire Line
+	6650 2350 6700 2350
 Wire Wire Line
 	7050 1950 7100 1950
@@
 	7100 2800 7100 3100
 Wire Wire Line
-	6900 3100 7150 3100
-$Comp
-L GND #PWR010
+	6900 3100 7100 3100
+$Comp
+L power:GND #PWR010
 U 1 1 5AC8103C
 P 6650 3200
@@
 $EndComp
 Wire Wire Line
-	6650 3200 7150 3200
+	6650 3200 6700 3200
 Wire Wire Line
 	6700 3200 6700 2800
@@
 Connection ~ 7100 3100
 $Comp
-L GND #PWR011
+L power:GND #PWR011
 U 1 1 5AC81356
 P 7000 3900
@@
 	7000 3900 7150 3900
 $Comp
-L GND #PWR012
+L power:GND #PWR012
 U 1 1 5AC81860
 P 7000 4550
@@
 	2600 3700 2900 3700
 $Comp
-L GND #PWR013
+L power:GND #PWR013
 U 1 1 5AC84E05
 P 4800 2500
@@
 	4700 2000 4700 2500
 Wire Wire Line
-	4350 2500 4800 2500
+	4350 2500 4700 2500
 Connection ~ 4700 2500
 $Comp
-L PWR_FLAG #FLG014
+L power:PWR_FLAG #FLG014
 U 1 1 5ACA03CA
 P 1250 900
@@
 SCL
 Wire Wire Line
-	6200 1150 7150 1150
-$Comp
-L ArduinoProMini U1
+	6200 1150 6550 1150
+$Comp
+L Homebrew:ArduinoProMini U1
 U 1 1 5AF60EC1
 P 1900 3100
@@
 NoConn ~ 2600 3800
 NoConn ~ 2600 3900
+Wire Wire Line
+	6550 950  7150 950
+Wire Wire Line
+	6550 1050 7150 1050
+Wire Wire Line
+	6550 1250 7150 1250
+Wire Wire Line
+	6550 1150 7150 1150
+Wire Wire Line
+	1050 3700 1150 3700
+Wire Wire Line
+	7100 2250 7150 2250
+Wire Wire Line
+	6700 2350 7150 2350
+Wire Wire Line
+	6700 3200 7150 3200
+Wire Wire Line
+	7100 3100 7150 3100
+Wire Wire Line
+	4700 2500 4800 2500
+Wire Wire Line
+	1250 900  1450 900
 $EndSCHEMATC
