File: HB-UNI-SEN-WEA/HB-UNI-SEN-WEA.sch (KiCad schematic (older format))
At the start: 17 parts, among them J1 PWR, J2 I2C_1, J3 I2C_2, J4 I2C_3, J5 ANEMOMETER, J6 RAIN_VOL, J7 WIND_DIR, J8 RAIN_SENS, J9 LIGHTNING, Q1 MPSA13, SW1 CONFIG_BUTTON, U1 ArduinoProMini, U2 CC1101

Commit message: * Switched to Kicad 5 * Added HB-UNI-644-S4-A4 addon Board
Parts:
- C1: symbol C_Small -> Device:C_Small
- C2: symbol CP_Small -> Device:CP_Small
- J1, J5, J6, J7: symbol Conn_01x02 -> conn:Conn_01x02
- J2, J3, J4, J8: symbol Conn_01x04 -> conn:Conn_01x04
- J9: symbol Conn_01x07 -> conn:Conn_01x07
- Q1: symbol Q_NPN_Darlington_EBC -> Device:Q_NPN_Darlington_EBC
- R1, R2: symbol R -> Device:R
- SW1: symbol SW_DIP_x01 -> switches:SW_DIP_x01
- U1: symbol ArduinoProMini -> Homebrew:ArduinoProMini
- U2: symbol CC1101 -> Homebrew:CC1101
Connections:
- wire segments 63 -> 74
Changed lines of the file:
@@
-EESchema Schematic File Version 2
-LIBS:HB-UNI-SEN-WEA-rescue
-LIBS:power
-LIBS:device
-LIBS:switches
-LIBS:relays
-LIBS:motors
-LIBS:transistors
-LIBS:conn
-LIBS:linear
-LIBS:regul
-LIBS:74xx
-LIBS:cmos4000
-LIBS:adc-dac
-LIBS:memory
-LIBS:xilinx
-LIBS:microcontrollers
-LIBS:dsp
-LIBS:microchip
-LIBS:analog_switches
-LIBS:motorola
-LIBS:texas
-LIBS:intel
-LIBS:audio
-LIBS:interface
-LIBS:digital-audio
-LIBS:philips
-LIBS:display
-LIBS:cypress
-LIBS:siliconi
-LIBS:opto
-LIBS:atmel
-LIBS:contrib
-LIBS:valves
-LIBS:Homebrew
+EESchema Schematic File Version 4
 LIBS:HB-UNI-SEN-WEA-cache
-EELAYER 25 0
+EELAYER 26 0
 EELAYER END
 $Descr A4 11693 8268
@@
 $EndDescr
 $Comp
-L Conn_01x04 J2
+L conn:Conn_01x04 J2
 U 1 1 5ABE0D25
 P 6750 1050
@@
 $EndComp
 $Comp
-L Conn_01x04 J3
+L conn:Conn_01x04 J3
 U 1 1 5ABE0DC1
 P 7350 1050
@@
 $EndComp
 $Comp
-L SW_DIP_x01 SW1
+L switches:SW_DIP_x01 SW1
 U 1 1 5ABE0E28
 P 4050 2500
@@
 $EndComp
 $Comp
-L Conn_01x02 J1
+L conn:Conn_01x02 J1
 U 1 1 5ABE2E32
 P 1650 900
@@
 $EndComp
 $Comp
-L GND #PWR01
+L power:GND #PWR01
 U 1 1 5AC7DE98
 P 6000 1050
@@
 $EndComp
 $Comp
-L GND #PWR02
+L power:GND #PWR02
 U 1 1 5AC7ECC2
 P 900 1000
@@
 $EndComp
 $Comp
-L GND #PWR03
+L power:GND #PWR03
 U 1 1 5AC7FA89
 P 1200 5900
@@
 $EndComp
 $Comp
-L GND #PWR04
+L power:GND #PWR04
 U 1 1 5AC7FD3C
 P 950 3750
@@
 $EndComp
 $Comp
-L GND #PWR05
+L power:GND #PWR05
 U 1 1 5AC81356
 P 6400 3150
@@
 $EndComp
 $Comp
-L GND #PWR06
+L power:GND #PWR06
 U 1 1 5AC84E05
 P 4800 2500
@@
 $EndComp
 $Comp
-L PWR_FLAG #FLG07
+L power:PWR_FLAG #FLG07
 U 1 1 5ACA03CA
 P 1250 900
@@
 SCL
 $Comp
-L ArduinoProMini U1
+L Homebrew:ArduinoProMini U1
 U 1 1 5AF60EC1
 P 1900 3100
@@
 D3
 $Comp
-L VCC #PWR08
+L power:VCC #PWR08
 U 1 1 5B60A376
 P 950 2000
@@
 $EndComp
 $Comp
-L VCC #PWR09
+L power:VCC #PWR09
 U 1 1 5B60A562
 P 900 900
@@
 $EndComp
 $Comp
-L +3.3V #PWR010
+L power:+3.3V #PWR010
 U 1 1 5B60A5AE
 P 1150 1900
@@
 $EndComp
 $Comp
-L +3.3V #PWR011
+L power:+3.3V #PWR011
 U 1 1 5B60A5E7
 P 1200 5350
@@
 $EndComp
 $Comp
-L +3.3V #PWR012
+L power:+3.3V #PWR012
 U 1 1 5B60A6DA
 P 6000 950
@@
 $EndComp
 $Comp
-L Conn_01x04 J4
+L conn:Conn_01x04 J4
 U 1 1 5B60A8CB
 P 7950 1050
@@
 $EndComp
 $Comp
-L Conn_01x02 J7
+L conn:Conn_01x02 J7
 U 1 1 5B60AC3C
 P 6750 3050
@@
 $EndComp
 $Comp
-L GND #PWR013
+L power:GND #PWR013
 U 1 1 5B60B1CC
 P 6400 2550
@@
 D6
 $Comp
-L Conn_01x02 J6
+L conn:Conn_01x02 J6
 U 1 1 5B60B1D5
 P 6750 2450
@@
 $EndComp
 $Comp
-L GND #PWR014
+L power:GND #PWR014
 U 1 1 5B60B27F
 P 6400 1950
@@
 D5
 $Comp
-L Conn_01x02 J5
+L conn:Conn_01x02 J5
 U 1 1 5B60B288
 P 6750 1850
@@
 $EndComp
 $Comp
-L Conn_01x04 J8
+L conn:Conn_01x04 J8
 U 1 1 5B60B45E
 P 8050 4200
@@
 $EndComp
 $Comp
-L VCC #PWR015
+L power:VCC #PWR015
 U 1 1 5B60B944
 P 7700 4100
@@
 $EndComp
 $Comp
-L GND #PWR016
+L power:GND #PWR016
 U 1 1 5B60BA08
 P 7700 4400
@@
 $EndComp
 $Comp
-L R R2
+L Device:R R2
 U 1 1 5B60BADF
 P 6900 4300
@@
 $EndComp
 $Comp
-L C_Small C1
+L Device:C_Small C1
 U 1 1 5B60BBC8
 P 7400 4300
@@
 D4
 $Comp
-L Q_NPN_Darlington_EBC Q1
+L Device:Q_NPN_Darlington_EBC Q1
 U 1 1 5B60C3E7
 P 7050 3800
@@
 $EndComp
 $Comp
-L GND #PWR017
+L power:GND #PWR017
 U 1 1 5B60C5F0
 P 6750 3900
@@
 $EndComp
 $Comp
-L R R1
+L Device:R R1
 U 1 1 5B60CA75
 P 6700 3600
@@
 D9
 $Comp
-L Conn_01x07 J9
+L conn:Conn_01x07 J9
 U 1 1 5B60CD7F
 P 7150 5250
@@
 Connection ~ 6550 1050
 Wire Wire Line
-	6200 1250 7750 1250
+	6200 1250 6550 1250
 Connection ~ 6550 1250
 Connection ~ 6550 1150
 Wire Wire Line
-	900  900  1450 900
+	900  900  1250 900
 Wire Wire Line
 	900  1000 1450 1000
@@
 	1200 5900 1350 5900
 Wire Wire Line
-	950  3700 1150 3700
+	950  3700 1050 3700
 Wire Wire Line
 	950  3750 950  3700
@@
 	6550 3050 6300 3050
 Wire Wire Line
-	6200 1150 7750 1150
+	6200 1150 6550 1150
 Wire Wire Line
 	2900 2000 2600 2000
@@
 	7850 4300 7500 4300
 Wire Wire Line
-	7300 4300 7050 4300
+	7300 4300 7150 4300
 Wire Wire Line
 	6300 4300 6750 4300
@@
 	7700 4400 7850 4400
 Wire Wire Line
-	6000 1050 7750 1050
-Wire Wire Line
-	6000 950  7750 950
-$Comp
-L GND #PWR018
+	6000 1050 6550 1050
+Wire Wire Line
+	6000 950  6550 950
+$Comp
+L power:GND #PWR018
 U 1 1 5B60D521
 P 6350 5050
@@
 $EndComp
 $Comp
-L +3.3V #PWR019
+L power:+3.3V #PWR019
 U 1 1 5B60D527
 P 6350 4950
@@
 NoConn ~ 2600 4100
 $Comp
-L CP_Small C2
+L Device:CP_Small C2
 U 1 1 5B60CD03
 P 1200 6650
@@
 $EndComp
 $Comp
-L +3.3V #PWR020
+L power:+3.3V #PWR020
 U 1 1 5B60CD87
 P 1200 6450
@@
 $EndComp
 $Comp
-L GND #PWR021
+L power:GND #PWR021
 U 1 1 5B60CDC5
 P 1200 6850
@@
 	1200 6750 1200 6850
 $Comp
-L CC1101 U2
+L Homebrew:CC1101 U2
 U 1 1 5B621728
 P 1650 5900
@@
 	1    0    0    -1
 $EndComp
+Wire Wire Line
+	6550 950  7150 950
+Wire Wire Line
+	6550 1050 7150 1050
+Wire Wire Line
+	6550 1250 7150 1250
+Wire Wire Line
+	6550 1150 7150 1150
+Wire Wire Line
+	1050 3700 1150 3700
+Wire Wire Line
+	1250 900  1450 900
+Wire Wire Line
+	7150 950  7750 950
+Wire Wire Line
+	7150 1050 7750 1050
+Wire Wire Line
+	7150 1150 7750 1150
+Wire Wire Line
+	7150 1250 7750 1250
+Wire Wire Line
+	7150 4300 7050 4300
 $EndSCHEMATC
